File: hardware design files/jlcpcb flex RF.kicad_sch (KiCad schematic)
At the start: 24 parts, among them J1 SMA, J10 SMA, J11 SMA, J12 SMA, J13 SMA, J14 SMA, J15 SMA, J16 SMA, J2 SMA, J3 SMA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

Commit message: Schematic Labeling
Other:
- title: (none) -> RF Charactarization
Changed lines of the file:
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@@
 	(generator_version "8.0")
 	(paper "A4")
+	(title_block
+		(title "RF Charactarization")
+		(date "2024-06-13")
+		(rev "A")
+	)
 	(junction
 		(at 129.54 50.8)
